Commit message: Add interactive URDF visualization with viser integration
- Add new visualization module with URDFVisualizer class
- Integrate viser library for web-based 3D robot visualization
- Add interactive joint control sliders and mesh display options
- Create command-line tools for hero visualization
- Fix OBJ file generation to remove problematic inline comments
- Add robust error handling and fallback visualization modes
- Update Hero class with visualize() method for easy access
- Add visualization dependencies as optional 'vis' extra
- Include comprehensive documentation and troubleshooting guide
- Add example scripts for complete visualization workflow

Features:
- Real-time joint manipulation via web interface
- Toggle visual/collision mesh display
- Automatic URDF loading with mesh path resolution
- Fallback modes for error recovery
- Cross-platform web-based interface

🤖 Generated with [Claude Code](https://claude.ai/code)

Co-Authored-By: Claude <noreply@anthropic.com>

File: heroes/tung_sahur_demo/robot.urdf (robot description, URDF)
Before this commit: robot tung_hero, 2 links, 1 joints
Links:
- added link chest_link, mass 0.1; collision box size=0.05 0.05 0.05; visual box size=0.05 0.05 0.05
- added link head_link, mass 0.1; collision box size=0.05 0.05 0.05; visual box size=0.05 0.05 0.05
- added link left_foot_link, mass 0.1; collision box size=0.05 0.05 0.05; visual box size=0.05 0.05 0.05
- added link left_hand_link, mass 0.1; collision box size=0.05 0.05 0.05; visual box size=0.05 0.05 0.05
- added link left_hip_link, mass 0.1; collision box size=0.05 0.05 0.05; visual box size=0.05 0.05 0.05
- added link left_lower_arm_link, mass 0.1; collision box size=0.05 0.05 0.05; visual box size=0.05 0.05 0.05
- added link left_lower_leg_link, mass 0.1; collision box size=0.05 0.05 0.05; visual box size=0.05 0.05 0.05
- added link left_shoulder_link, mass 0.1; collision box size=0.05 0.05 0.05; visual box size=0.05 0.05 0.05
- added link left_upper_arm_link, mass 0.1; collision box size=0.05 0.05 0.05; visual box size=0.05 0.05 0.05
- added link left_upper_leg_link, mass 0.1; collision box size=0.05 0.05 0.05; visual box size=0.05 0.05 0.05
- added link neck_link, mass 0.1; collision box size=0.05 0.05 0.05; visual box size=0.05 0.05 0.05
- added link right_foot_link, mass 0.1; collision box size=0.05 0.05 0.05; visual box size=0.05 0.05 0.05
- added link right_hand_link, mass 0.1; collision box size=0.05 0.05 0.05; visual box size=0.05 0.05 0.05
- added link right_hip_link, mass 0.1; collision box size=0.05 0.05 0.05; visual box size=0.05 0.05 0.05
- added link right_lower_arm_link, mass 0.1; collision box size=0.05 0.05 0.05; visual box size=0.05 0.05 0.05
- added link right_lower_leg_link, mass 0.1; collision box size=0.05 0.05 0.05; visual box size=0.05 0.05 0.05
- added link right_shoulder_link, mass 0.1; collision box size=0.05 0.05 0.05; visual box size=0.05 0.05 0.05
- added link right_upper_arm_link, mass 0.1; collision box size=0.05 0.05 0.05; visual box size=0.05 0.05 0.05
- added link right_upper_leg_link, mass 0.1; collision box size=0.05 0.05 0.05; visual box size=0.05 0.05 0.05
- added link spine_link, mass 0.1; collision box size=0.05 0.05 0.05; visual box size=0.05 0.05 0.05
Joints:
- added joint chest_to_left_shoulder: type revolute, parent chest_link, child left_shoulder_link, origin xyz=-0.200 1.300 0.000 rpy=0 0 0, axis 0 0 1, limit lower=-3.14159 upper=3.14159 effort=100 velocity=10
- added joint chest_to_neck: type revolute, parent chest_link, child neck_link, origin xyz=0.000 1.500 0.000 rpy=0 0 0, axis 0 0 1, limit lower=-3.14159 upper=3.14159 effort=100 velocity=10
- added joint chest_to_right_shoulder: type revolute, parent chest_link, child right_shoulder_link, origin xyz=0.200 1.300 0.000 rpy=0 0 0, axis 0 0 1, limit lower=-3.14159 upper=3.14159 effort=100 velocity=10
- added joint left_hip_to_left_upper_leg: type revolute, parent left_hip_link, child left_upper_leg_link, origin xyz=-0.100 0.400 0.000 rpy=0 0 0, axis 0 0 1, limit lower=-3.14159 upper=3.14159 effort=100 velocity=10
- added joint left_lower_arm_to_left_hand: type revolute, parent left_lower_arm_link, child left_hand_link, origin xyz=-0.300 0.400 0.000 rpy=0 0 0, axis 0 0 1, limit lower=-3.14159 upper=3.14159 effort=100 velocity=10
- added joint left_lower_leg_to_left_foot: type revolute, parent left_lower_leg_link, child left_foot_link, origin xyz=-0.100 -0.300 0.000 rpy=0 0 0, axis 0 0 1, limit lower=-3.14159 upper=3.14159 effort=100 velocity=10
- added joint left_shoulder_to_left_upper_arm: type revolute, parent left_shoulder_link, child left_upper_arm_link, origin xyz=-0.300 1.100 0.000 rpy=0 0 0, axis 0 0 1, limit lower=-3.14159 upper=3.14159 effort=100 velocity=10
- added joint left_upper_arm_to_left_lower_arm: type revolute, parent left_upper_arm_link, child left_lower_arm_link, origin xyz=-0.300 0.700 0.000 rpy=0 0 0, axis 0 0 1, limit lower=-3.14159 upper=3.14159 effort=100 velocity=10
- added joint left_upper_leg_to_left_lower_leg: type revolute, parent left_upper_leg_link, child left_lower_leg_link, origin xyz=-0.100 0.000 0.000 rpy=0 0 0, axis 0 0 1, limit lower=-3.14159 upper=3.14159 effort=100 velocity=10
- added joint neck_to_head: type revolute, parent neck_link, child head_link, origin xyz=0.000 1.700 0.000 rpy=0 0 0, axis 0 0 1, limit lower=-3.14159 upper=3.14159 effort=100 velocity=10
- added joint pelvis_to_left_hip: type revolute, parent pelvis_link, child left_hip_link, origin xyz=-0.100 0.700 0.000 rpy=0 0 0, axis 0 0 1, limit lower=-3.14159 upper=3.14159 effort=100 velocity=10
- added joint pelvis_to_right_hip: type revolute, parent pelvis_link, child right_hip_link, origin xyz=0.100 0.700 0.000 rpy=0 0 0, axis 0 0 1, limit lower=-3.14159 upper=3.14159 effort=100 velocity=10
- added joint pelvis_to_spine: type revolute, parent pelvis_link, child spine_link, origin xyz=0.000 1.000 0.000 rpy=0 0 0, axis 0 0 1, limit lower=-3.14159 upper=3.14159 effort=100 velocity=10
- added joint right_hip_to_right_upper_leg: type revolute, parent right_hip_link, child right_upper_leg_link, origin xyz=0.100 0.400 0.000 rpy=0 0 0, axis 0 0 1, limit lower=-3.14159 upper=3.14159 effort=100 velocity=10
- added joint right_lower_arm_to_right_hand: type revolute, parent right_lower_arm_link, child right_hand_link, origin xyz=0.300 0.400 0.000 rpy=0 0 0, axis 0 0 1, limit lower=-3.14159 upper=3.14159 effort=100 velocity=10
- added joint right_lower_leg_to_right_foot: type revolute, parent right_lower_leg_link, child right_foot_link, origin xyz=0.100 -0.300 0.000 rpy=0 0 0, axis 0 0 1, limit lower=-3.14159 upper=3.14159 effort=100 velocity=10
- added joint right_shoulder_to_right_upper_arm: type revolute, parent right_shoulder_link, child right_upper_arm_link, origin xyz=0.300 1.100 0.000 rpy=0 0 0, axis 0 0 1, limit lower=-3.14159 upper=3.14159 effort=100 velocity=10
- added joint right_upper_arm_to_right_lower_arm: type revolute, parent right_upper_arm_link, child right_lower_arm_link, origin xyz=0.300 0.700 0.000 rpy=0 0 0, axis 0 0 1, limit lower=-3.14159 upper=3.14159 effort=100 velocity=10
- added joint right_upper_leg_to_right_lower_leg: type revolute, parent right_upper_leg_link, child right_lower_leg_link, origin xyz=0.100 0.000 0.000 rpy=0 0 0, axis 0 0 1, limit lower=-3.14159 upper=3.14159 effort=100 velocity=10
- added joint spine_to_chest: type revolute, parent spine_link, child chest_link, origin xyz=0.000 1.200 0.000 rpy=0 0 0, axis 0 0 1, limit lower=-3.14159 upper=3.14159 effort=100 velocity=10
